File: gps-seven-seg-clock.kicad_pcb (KiCad board)
At the start: 2 copper layers, 14 parts, among them U1 ATmega328PB-A, U2 MAX-M10S

Commit message: finished
Parts:
- removed AFF1, AFF2, AFF3, AFF4, AFF5, AFF6: LTS-6960HR, Display_7Segment:7SegmentLED_LTS6760_LTS6780
- removed D4, D5: LED, LED_THT:LED_D5.0mm
- removed PS1: IRM-20-3.3, Converter_ACDC:Converter_ACDC_MeanWell_IRM-20-xx_THT
- added C1: 0.1uF, Capacitor_SMD:C_0603_1608Metric, F.Cu at (129.8, 44.4)
- added C10: 0.1uF, Capacitor_SMD:C_0603_1608Metric, F.Cu at (103.2, 41.6)
- added C11: 0.1uF, Capacitor_SMD:C_0603_1608Metric, F.Cu at (117.4, 66.8)
- added C12: 10uF, Capacitor_SMD:C_0603_1608Metric, F.Cu at (119.2, 66.8)
- added C13: 0.1uF, Capacitor_SMD:C_0603_1608Metric, F.Cu at (161.2, 44.4)
- added C14: 10uF, Capacitor_SMD:C_0603_1608Metric, F.Cu at (120.0, 50.2)
- added C15: 0.1uF, Capacitor_SMD:C_0603_1608Metric, F.Cu at (114.8, 59.6)
- added C16: 0.1uF, Capacitor_SMD:C_0603_1608Metric, F.Cu at (128.8, 56.4)
- added C17: 0.1uF, Capacitor_SMD:C_0603_1608Metric, F.Cu at (125.2, 48.2)
- added C2: 0.1uF, Capacitor_SMD:C_0603_1608Metric, F.Cu at (81.2, 40.8)
- added C3: 10nF, Capacitor_SMD:C_0603_1608Metric, F.Cu at (96.2, 40.8)
- added C4: 10uF, Capacitor_SMD:C_0603_1608Metric, F.Cu at (112.2, 46.0)
- added C5: 0.1uF, Capacitor_SMD:C_0603_1608Metric, F.Cu at (113.6, 32.8)
- added C6: 0.1uF, Capacitor_SMD:C_0603_1608Metric, F.Cu at (145.6, 44.4)
- added C7: 100uF, Capacitor_SMD:CP_Elec_6.3x5.4_Nichicon, F.Cu at (97.2, 55.0)
- added C8: 0.1uF, Capacitor_SMD:C_0603_1608Metric, F.Cu at (112.8, 63.2)
- added C9: 0.1uF, Capacitor_SMD:C_0603_1608Metric, F.Cu at (120.4, 35.0)
- added H1: M3, MountingHole:MountingHole_3.2mm_M3, F.Cu at (176.6, 28.4)
- added H2: M3, MountingHole:MountingHole_3.2mm_M3, F.Cu at (176.6, 71.6)
- added H3: M3, MountingHole:MountingHole_3.2mm_M3, F.Cu at (83.4, 28.4)
- added H4: M3, MountingHole:MountingHole_3.2mm_M3, F.Cu at (83.4, 71.6)
- added J1: SMA, Connector_Coaxial:SMA_Amphenol_132289_EdgeMount, F.Cu at (97.0, 27.8)
- added J10: SM09B-GHS-TB, Connector_JST:JST_GH_SM09B-GHS-TB_1x09-1MP_P1.25mm_Horizontal, F.Cu at (147.2, 71.8)
- added J11: SM09B-GHS-TB, Connector_JST:JST_GH_SM09B-GHS-TB_1x09-1MP_P1.25mm_Horizontal, F.Cu at (147.0, 28.2)
- added J12: SM04B-GHS-TB, Connector_JST:JST_GH_SM04B-GHS-TB_1x04-1MP_P1.25mm_Horizontal, F.Cu at (176.6, 49.1)
- added J2: SM09B-GHS-TB, Connector_JST:JST_GH_SM09B-GHS-TB_1x09-1MP_P1.25mm_Horizontal, F.Cu at (131.2, 71.8)
- added J3: SM09B-GHS-TB, Connector_JST:JST_GH_SM09B-GHS-TB_1x09-1MP_P1.25mm_Horizontal, F.Cu at (131.1, 28.2)
- added J4: ICSP, Connector_PinSocket_2.00mm:PinSocket_2x03_P2.00mm_Vertical, F.Cu at (117.0, 27.0)
- added J5: XT30PW-M, Connector_AMASS:AMASS_XT30PW-M_1x02_P2.50mm_Horizontal, F.Cu at (93.1, 61.3)
- added J6: SM04B-GHS-TB, Connector_JST:JST_GH_SM04B-GHS-TB_1x04-1MP_P1.25mm_Horizontal, F.Cu at (109.6, 28.2)
- added J7: SM09B-GHS-TB, Connector_JST:JST_GH_SM09B-GHS-TB_1x09-1MP_P1.25mm_Horizontal, F.Cu at (163.1, 71.8)
- added J8: SM09B-GHS-TB, Connector_JST:JST_GH_SM09B-GHS-TB_1x09-1MP_P1.25mm_Horizontal, F.Cu at (162.9, 28.2)
- added J9: SM06B-GHS-TB, Connector_JST:JST_GH_SM06B-GHS-TB_1x06-1MP_P1.25mm_Horizontal, F.Cu at (83.2, 59.2)
- added L1: 2.66, Inductor_SMD:L_0805_2012Metric_Pad1.15x1.40mm_HandSolder, F.Cu at (97.0, 35.6)
- added Q2: MJD127, Package_TO_SOT_SMD:TO-252-2, F.Cu at (122.4, 59.0)
- added R1: 10, Resistor_SMD:R_0603_1608Metric, F.Cu at (96.2, 38.8)
- added R10: 100K, Resistor_SMD:R_0603_1608Metric, F.Cu at (120.4, 37.4)
- added R11: 10K, Resistor_SMD:R_0603_1608Metric, F.Cu at (116.4, 50.2)
- added R12: 4.99K, Resistor_SMD:R_0603_1608Metric, F.Cu at (110.8, 59.6)
- added R13: 470, Resistor_SMD:R_1206_3216Metric, F.Cu at (174.7, 40.3)
- added R14: 1K, Resistor_SMD:R_0603_1608Metric, F.Cu at (124.0, 50.2)
- added R15: 1K, Resistor_SMD:R_0603_1608Metric, F.Cu at (127.0, 56.4)
- added R16: 10K, Resistor_SMD:R_0603_1608Metric, F.Cu at (127.0, 53.0)
- added R17: 470, Resistor_SMD:R_1206_3216Metric, F.Cu at (174.5, 57.6)
- added R2: 2.2K, Resistor_SMD:R_0603_1608Metric, F.Cu at (103.2, 35.4)
- added R3: 2.2K, Resistor_SMD:R_0603_1608Metric, F.Cu at (103.2, 37.5)
- added R4: 2.2K, Resistor_SMD:R_0603_1608Metric, F.Cu at (157.7, 50.6)
- added R5: 2.2K, Resistor_SMD:R_0603_1608Metric, F.Cu at (157.7, 48.2)
- added R6: 100K, Resistor_SMD:R_0603_1608Metric, F.Cu at (103.2, 39.6)
- added R7: 1K, Resistor_SMD:R_0603_1608Metric, F.Cu at (120.4, 39.6)
- added R8: 100K, Resistor_SMD:R_0603_1608Metric, F.Cu at (110.2, 32.8)
- added R9: 100K, Resistor_SMD:R_0603_1608Metric, F.Cu at (106.6, 32.8)
- added SW1: 219-2LPST, Button_Switch_SMD:SW_DIP_SPSTx02_Slide_6.7x6.64mm_W8.61mm_P2.54mm_LowProfile, F.Cu at (86.4, 48.6)
- added TP1: 5016, jannett_footprints:TestPoint_Keystone_5016_Vias, F.Cu at (120.0, 72.2)
- added TP2: 5016, jannett_footprints:TestPoint_Keystone_5016_Vias, F.Cu at (106.0, 54.0)
- added TP3: 5016, jannett_footprints:TestPoint_Keystone_5016_Vias, F.Cu at (106.0, 72.2)
- added TP4: 5016, jannett_footprints:TestPoint_Keystone_5016_Vias, F.Cu at (106.0, 60.6)
- added U10: AD8676xR, Package_SO:SOIC-8_3.9x4.9mm_P1.27mm, F.Cu at (113.6, 55.0)
- added U11: PCA9555PW, Package_SO:TSSOP-24_4.4x7.8mm_P0.65mm, F.Cu at (148.3, 49.4)
- added U12: ULN2003A, Package_SO:SOIC-16_3.9x9.9mm_P1.27mm, F.Cu at (147.7, 63.7)
- added U13: ULN2003A, Package_SO:SOIC-16_3.9x9.9mm_P1.27mm, F.Cu at (146.4, 36.8)
- added U3: ULN2003A, Package_SO:SOIC-16_3.9x9.9mm_P1.27mm, F.Cu at (131.9, 63.7)
- added U4: ULN2003A, Package_SO:SOIC-16_3.9x9.9mm_P1.27mm, F.Cu at (130.4, 36.8)
- added U5: ATmega328PB-A, Package_QFP:TQFP-32_7x7mm_P0.8mm, F.Cu at (112.4, 39.4)
- added U6: PCA9555PW, Package_SO:TSSOP-24_4.4x7.8mm_P0.65mm, F.Cu at (163.9, 49.3)
- added U7: ULN2003A, Package_SO:SOIC-16_3.9x9.9mm_P1.27mm, F.Cu at (163.8, 63.6)
- added U8: ULN2003A, Package_SO:SOIC-16_3.9x9.9mm_P1.27mm, F.Cu at (162.4, 36.7)
- added U9: NCP1117-3.3_TO252, Package_TO_SOT_SMD:TO-252-2, F.Cu at (112.7, 69.8)
- added Y1: 8MHz, Crystal:Resonator_SMD_Murata_CSTxExxV-3Pin_3.0x1.1mm_HandSoldering, F.Cu at (120.4, 45.0)
- D1: value SFH203 -> LED; footprint LED_THT:LED_D5.0mm_IRGrey -> LED_SMD:LED_0603_1608Metric_Pad1.05x0.95mm_HandSolder
- D2, D3: value LED -> B5819W; footprint LED_THT:LED_D5.0mm -> Diode_SMD:D_SOD-123
- U1: value ATmega328PB-A -> PCA9555PW; footprint Package_QFP:TQFP-32_7x7mm_P0.8mm -> Package_SO:TSSOP-24_4.4x7.8mm_P0.65mm
- moved D3 75.5 mm to (89.2, 57.2), turned to 180 degrees
- moved U2 68.0 mm to (88.2, 38.8)
- moved D1 58.2 mm to (120.5, 41.7)
- moved D2 52.1 mm to (106.0, 66.2), turned to -90 degrees
- moved U1 37.2 mm to (132.4, 49.5), turned to 90 degrees
Connections:
- D1 pad 1: unconnected-(D1-K-Pad1) -> GND
- D1 pad 2: unconnected-(D1-A-Pad2) -> Net-(D1-A)
- D2 pad 1: unconnected-(D2-K-Pad1) -> +12V
- D2 pad 2: unconnected-(D2-A-Pad2) -> +3.3V
- D3 pad 1: unconnected-(D3-K-Pad1) -> +12V
- D3 pad 2: unconnected-(D3-A-Pad2) -> Net-(D3-A)
- U1 pad 10: unconnected-(U1-PD6-Pad10) -> Net-(U1-IO0_6)
- U1 pad 12: unconnected-(U1-PB0-Pad12) -> GND
- U1 pad 13: unconnected-(U1-PB1-Pad13) -> Net-(U1-IO1_0)
- U1 pad 14: unconnected-(U1-PB2-Pad14) -> Net-(U1-IO1_1)
- U1 pad 15: unconnected-(U1-PB3-Pad15) -> Net-(U1-IO1_2)
- U1 pad 16: unconnected-(U1-PB4-Pad16) -> Net-(U1-IO1_3)
- U1 pad 17: unconnected-(U1-PB5-Pad17) -> Net-(U1-IO1_4)
- U1 pad 18: unconnected-(U1-AVCC-Pad18) -> Net-(U1-IO1_5)
- U1 pad 19: unconnected-(U1-PE2-Pad19) -> Net-(U1-IO1_6)
- U1 pad 2: unconnected-(U1-PD4-Pad2) -> GND
- U1 pad 21: Net-(U1-GND-Pad21) -> GND
- U1 pad 22: unconnected-(U1-PE3-Pad22) -> /SCL1
- U1 pad 23: unconnected-(U1-PC0-Pad23) -> /SDA1
- U1 pad 24: unconnected-(U1-PC1-Pad24) -> +3.3V
- U1 pad 3: unconnected-(U1-PE0-Pad3) -> GND
- U1 pad 4: unconnected-(U1-VCC-Pad4) -> Net-(U1-IO0_0)
- U1 pad 5: Net-(U1-GND-Pad21) -> Net-(U1-IO0_1)
- U1 pad 6: unconnected-(U1-PE1-Pad6) -> Net-(U1-IO0_2)
- U1 pad 7: unconnected-(U1-XTAL1/PB6-Pad7) -> Net-(U1-IO0_3)
- U1 pad 8: unconnected-(U1-XTAL2/PB7-Pad8) -> Net-(U1-IO0_4)
- U1 pad 9: unconnected-(U1-PD5-Pad9) -> Net-(U1-IO0_5)
- U2 pad 1: Net-(U2-GND-Pad1) -> GND
- U2 pad 10: Net-(U2-GND-Pad1) -> GND
- U2 pad 11: unconnected-(U2-RF_IN-Pad11) -> Net-(J1-In)
- U2 pad 12: Net-(U2-GND-Pad1) -> GND
- U2 pad 14: unconnected-(U2-VCC_RF-Pad14) -> Net-(U2-VCC_RF)
- U2 pad 16: unconnected-(U2-SDA-Pad16) -> /SDA
- U2 pad 17: unconnected-(U2-SCL-Pad17) -> /SCL
- U2 pad 2: unconnected-(U2-TXD-Pad2) -> /GPS_TX
- U2 pad 3: unconnected-(U2-RXD-Pad3) -> /GPS_RX
- U2 pad 4: unconnected-(U2-TIMEPULSE-Pad4) -> /PPS
- U2 pad 6: unconnected-(U2-V_BCKP-Pad6) -> +3.3V
- U2 pad 7: unconnected-(U2-VCC_IO-Pad7) -> +3.3V
- U2 pad 8: unconnected-(U2-VCC-Pad8) -> +3.3V
Routing:
- net GND: track 0.00 -> 75.4 mm, vias 0 -> 97
- net /SCL1: track 0.00 -> 64.2 mm, vias 0 -> 4
- net /SDA1: track 0.00 -> 64.0 mm, vias 0 -> 4
- net +3.3V: track 0.00 -> 49.3 mm, vias 0 -> 11
- net /TX: track 0.00 -> 40.2 mm, vias 0 -> 3
- net Net-(J9-Pin_3): track 0.00 -> 39.0 mm, vias 0 -> 2
- net /RX: track 0.00 -> 38.6 mm, vias 0 -> 3
- net /SCL: track 0.00 -> 38.0 mm, vias 0 -> 2
- net /SDA: track 0.00 -> 37.3 mm, vias 0 -> 2
- net /PPS: track 0.00 -> 34.2 mm, vias 0 -> 2
- net /RESET: track 0.00 -> 30.6 mm, vias 0 -> 1
- net Net-(U10A-+): track 0.00 -> 28.7 mm
- net VDD: track 0.00 -> 25.9 mm, vias 0 -> 14
- net Net-(U10B-+): track 0.00 -> 25.5 mm, vias 0 -> 2
- net Net-(J1-In): track 0.00 -> 24.9 mm
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- added copper zone on B.Cu, net +12V
- added copper zone on F.Cu, net +12V
- added copper zone on In2.Cu, net +12V
- added copper zone on F.Cu, net +3.3V
- added copper zone on In2.Cu, net +3.3V
- added copper zone on B.Cu, net GND
- added copper zone on F.Cu, net GND
- added copper zone on In1.Cu, net GND
- added copper zone on In2.Cu, net GND
- added copper zone on B.Cu, net VDD
- added copper zone on F.Cu, net VDD
- added copper zone on In2.Cu, net VDD
Other:
- board outline added: 100 x 50 mm
- copper layers 2 -> 4
- board text added: "1 3.3V 2 VIN 3 RST 4 RX 5 TX 6 GND"
- board text added: "1,2 Anodes 3-9 Cathodes"
- board text added: "12V"
- board text added: "3.3V"
- board text added: "4 GND 3 A1 2 GND 1 A0"
- board text added: "4 GND 3 Anode 2 GND 1 Anode"
- board text added: "Anode"
- board text added: "GND"
- board text added: "GPS Antenna"
- board text added: "GPS Clock"
- board text added: "Jannett W"
- board text added: "MISO"
- board text added: "MOSI"
- board text added: "RST"
- board text added: "RX"
- board text added: "SCK"
- board text added: "TX"
