File: gps-seven-seg-clock.kicad_sch (KiCad schematic)
At the start: 15 parts, among them U1 ATmega328PB-A, U2 MAX-M10S, Y1 Crystal_GND2_Small

Commit message: finished
Parts:
- removed AFF1, AFF2, AFF3, AFF4, AFF5, AFF6: LTS-6960HR, Display_7Segment:7SegmentLED_LTS6760_LTS6780, symbol Display_Character:LTS-6960HR
- removed D1: SFH203, LED_THT:LED_D5.0mm_IRGrey, symbol Sensor_Optical:SFH203
- removed D2, D3, D4, D5: LED, LED_THT:LED_D5.0mm, symbol Device:LED
- removed PS1: IRM-20-3.3, Converter_ACDC:Converter_ACDC_MeanWell_IRM-20-xx_THT, symbol Converter_ACDC:IRM-20-3.3
- added C1, C10, C11, C13, C15, C16, C17, C2, C5, C6, C8, C9: 0.1uF, Capacitor_SMD:C_0603_1608Metric, symbol Device:C_Small
- added C12, C14, C4: 10uF, Capacitor_SMD:C_0603_1608Metric, symbol Device:C_Small
- added C3: 10nF, Capacitor_SMD:C_0603_1608Metric, symbol Device:C_Small
- added C7: 100uF, Capacitor_SMD:CP_Elec_6.3x5.4_Nichicon, symbol Device:C_Polarized_US
- added D1: LED, LED_SMD:LED_0603_1608Metric_Pad1.05x0.95mm_HandSolder, symbol Device:LED
- added D2, D3: B5819W, Diode_SMD:D_SOD-123, symbol Device:D_Schottky
- added H1, H2, H3, H4: M3, MountingHole:MountingHole_3.2mm_M3, symbol Mechanical:MountingHole
- added J1: SMA, Connector_Coaxial:SMA_Amphenol_132289_EdgeMount, symbol Connector:Conn_Coaxial
- added J10, J11, J2, J3, J7, J8: SM09B-GHS-TB, Connector_JST:JST_GH_SM09B-GHS-TB_1x09-1MP_P1.25mm_Horizontal, symbol Connector_Generic:Conn_01x09
- added J12, J6: SM04B-GHS-TB, Connector_JST:JST_GH_SM04B-GHS-TB_1x04-1MP_P1.25mm_Horizontal, symbol Connector_Generic:Conn_01x04
- added J4: ICSP, Connector_PinSocket_2.00mm:PinSocket_2x03_P2.00mm_Vertical, symbol Connector_Generic:Conn_02x03_Odd_Even
- added J5: XT30PW-M, Connector_AMASS:AMASS_XT30PW-M_1x02_P2.50mm_Horizontal, symbol Connector_Generic:Conn_01x02
- added J9: SM06B-GHS-TB, Connector_JST:JST_GH_SM06B-GHS-TB_1x06-1MP_P1.25mm_Horizontal, symbol Connector_Generic:Conn_01x06
- added L1: 2.66, Inductor_SMD:L_0805_2012Metric_Pad1.15x1.40mm_HandSolder, symbol Device:L_Ferrite_Small
- added Q2: MJD127, Package_TO_SOT_SMD:TO-252-2, symbol Transistor_BJT:Q_PNP_Darlington_BCE
- added R1: 10, Resistor_SMD:R_0603_1608Metric, symbol Device:R_US
- added R10, R6, R8, R9: 100K, Resistor_SMD:R_0603_1608Metric, symbol Device:R_US
- added R11, R16: 10K, Resistor_SMD:R_0603_1608Metric, symbol Device:R_US
- added R12: 4.99K, Resistor_SMD:R_0603_1608Metric, symbol Device:R_US
- added R13, R17: 470, Resistor_SMD:R_1206_3216Metric, symbol Device:R_US
- added R14, R15, R7: 1K, Resistor_SMD:R_0603_1608Metric, symbol Device:R_US
- added R2, R3, R4, R5: 2.2K, Resistor_SMD:R_0603_1608Metric, symbol Device:R_US
- added SW1: 219-2LPST, Button_Switch_SMD:SW_DIP_SPSTx02_Slide_6.7x6.64mm_W8.61mm_P2.54mm_LowProfile, symbol Switch:SW_DIP_x02
- added TP1, TP2, TP3, TP4: 5016, jannett_footprints:TestPoint_Keystone_5016_Vias, symbol Connector:TestPoint
- added U1, U11, U6: PCA9555PW, Package_SO:TSSOP-24_4.4x7.8mm_P0.65mm, symbol Interface_Expansion:PCA9555PW
- added U10: AD8676xR, Package_SO:SOIC-8_3.9x4.9mm_P1.27mm, symbol Amplifier_Operational:AD8676xR
- added U12, U13, U3, U4, U7, U8: ULN2003A, Package_SO:SOIC-16_3.9x9.9mm_P1.27mm, symbol Transistor_Array:ULN2003A
- added U9: NCP1117-3.3_TO252, Package_TO_SOT_SMD:TO-252-2, symbol Regulator_Linear:NCP1117-3.3_TO252
- Y1: value Crystal_GND2_Small -> 8MHz; footprint (none) -> Crystal:Resonator_SMD_Murata_CSTxExxV-3Pin_3.0x1.1mm_HandSoldering
- renumbered U1 to U5
Connections:
- net at Y1.1: now also U5.7 (XTAL1/PB6)
- net GND: now reaches Y1.2
- net GND: now also U2.1 (GND), U2.10 (GND), U2.12 (GND), U5.21 (GND), U5.5 (GND), C1.2, C11.2, C12.2, C13.2, C14.2, C15.2, C16.2, C2.2, C3.2, C4.2, C5.2, C6.2, C7.2, C8.2, C9.2, D1.1 (K), J1.2 (Ext), J12.2 (Pin_2), J12.4 (Pin_4), J4.6 (Pin_6), J5.2 (Pin_2), J6.2 (Pin_2), J6.4 (Pin_4), J9.6 (Pin_6), R16.2, TP2.1, U1.12 (VSS), U1.2 (A1), U1.21 (A0), U1.3 (A2), U10.4 (V-), U11.12 (VSS), U11.21 (A0), U11.3 (A2), U12.8 (GND), U13.8 (GND), U3.8 (GND), U4.8 (GND), U6.12 (VSS), U6.2 (A1), U6.3 (A2), U7.8 (GND), U8.8 (GND), U9.1 (GND)
- net at Y1.3: now also U5.8 (XTAL2/PB7)
- net at U2.11 (RF_IN): now also J1.1 (In), L1.2
- net at U2.14 (VCC_RF): now also R1.1
- net SDA: now reaches U2.16 (SDA)
- net SDA: now also U5.27 (PC4), R2.2
- net SCL: now reaches U2.17 (SCL)
- net SCL: now also U5.28 (PC5), R3.2
- net GPS_TX: now reaches U2.2 (TXD)
- net GPS_TX: now also SW1.3
- net GPS_RX: now reaches U2.3 (RXD)
- net GPS_RX: now also SW1.4
- net PPS: now reaches U2.4 (TIMEPULSE)
- net PPS: now also U5.1 (PD3)
- net +3.3V: now reaches U2.6 (V_BCKP)
- net +3.3V: now also U2.7 (VCC_IO), U2.8 (VCC), U5.18 (AVCC), U5.4 (VCC), C1.1, C11.1, C12.1, C13.1, C2.1, C4.1, C5.1, C6.1, D2.2 (A), J4.2 (Pin_2), J9.1 (Pin_1), R2.1, R3.1, R4.1, R5.1, R6.2, R8.2, R9.2, TP3.1, U1.24 (VDD), U11.2 (A1), U11.24 (VDD), U6.21 (A0), U6.24 (VDD), U9.2 (VO)
- net LED_INT: now reaches U5.11 (PD7)
- net LED_INT: now also R7.1
- net PWM9: now reaches U5.13 (PB1)
- net PWM9: now also R10.1
- net MOSI: now reaches U5.15 (PB3)
- net MOSI: now also J4.4 (Pin_4)
- net MISO: now reaches U5.16 (PB4)
- net MISO: now also J4.1 (Pin_1)
- net SCK: now reaches U5.17 (PB5)
- net SCK: now also J4.3 (Pin_3)
- net ADC0: now reaches U5.23 (PC0)
- net ADC0: now also J6.1 (Pin_1), R8.1
- net ADC1: now reaches U5.24 (PC1)
- net ADC1: now also J6.3 (Pin_3), R9.1
- net RESET: now reaches U5.29 (~{RESET}/PC6)
- net RESET: now also C10.1, J4.5 (Pin_5), R6.1
- net SDA1: now reaches U5.3 (PE0)
- net SDA1: now also R5.2, U1.23 (SDA), U11.23 (SDA), U6.23 (SDA)
- net RX: now reaches U5.30 (PD0)
- net RX: now also J9.4 (Pin_4), SW1.1
- net TX: now reaches U5.31 (PD1)
- net TX: now also J9.5 (Pin_5), SW1.2
- net SCL1: now reaches U5.6 (PE1)
- net SCL1: now also R4.2, U1.22 (SCL), U11.22 (SCL), U6.22 (SCL)
- new net: C16.1, R15.1, R16.1, U10.5 (+)
- new net: U1.10 (IO0_6), U3.1 (I1)
- new net: U1.9 (IO0_5), U3.2 (I2)
- new net: U1.8 (IO0_4), U3.3 (I3)
- new net: U1.7 (IO0_3), U3.4 (I4)
- new net: U1.6 (IO0_2), U3.5 (I5)
- new net: U1.5 (IO0_1), U3.6 (I6)
- new net: U1.4 (IO0_0), U3.7 (I7)
- new net: R11.1, U10.1, U10.2 (-)
- new net: C14.1, C17.2, R11.2, R12.1, U10.6 (-)
- new net: C3.1, L1.1, R1.2
- new net: C17.1, R14.1, U10.7
- new net: U6.19 (IO1_6), U8.1 (I1)
- new net: U6.18 (IO1_5), U8.2 (I2)
- new net: U6.17 (IO1_4), U8.3 (I3)
- new net: U6.16 (IO1_3), U8.4 (I4)
- new net: U6.15 (IO1_2), U8.5 (I5)
- new net: U6.14 (IO1_1), U8.6 (I6)
- new net: U6.13 (IO1_0), U8.7 (I7)
- new net: C9.1, R10.2, U10.3 (+)
- new net: Q2.1 (B), R14.2
- new net: U6.10 (IO0_6), U7.1 (I1)
- new net: U6.4 (IO0_0), U7.7 (I7)
- new net: U6.5 (IO0_1), U7.6 (I6)
- new net: U6.6 (IO0_2), U7.5 (I5)
- new net: U6.7 (IO0_3), U7.4 (I4)
- new net: U6.8 (IO0_4), U7.3 (I3)
- new net: U6.9 (IO0_5), U7.2 (I2)
- new net: J12.1 (Pin_1), R17.2
- new net: D3.2 (A), J9.2 (Pin_2)
- new net: C10.2, J9.3 (Pin_3)
- new net: D1.2 (A), R7.2
- new net: U1.19 (IO1_6), U4.1 (I1)
- new net: U1.18 (IO1_5), U4.2 (I2)
- new net: U1.17 (IO1_4), U4.3 (I3)
- new net: U1.16 (IO1_3), U4.4 (I4)
- new net: U1.15 (IO1_2), U4.5 (I5)
- new net: U1.14 (IO1_1), U4.6 (I6)
- new net: U1.13 (IO1_0), U4.7 (I7)
- new net: U11.10 (IO0_6), U12.1 (I1)
- new net: U11.9 (IO0_5), U12.2 (I2)
- new net: U11.8 (IO0_4), U12.3 (I3)
- new net: U11.7 (IO0_3), U12.4 (I4)
- new net: U11.6 (IO0_2), U12.5 (I5)
- new net: U11.5 (IO0_1), U12.6 (I6)
- new net: U11.4 (IO0_0), U12.7 (I7)
- new net: J12.3 (Pin_3), R13.2
- new net: U11.19 (IO1_6), U13.1 (I1)
- new net: U11.18 (IO1_5), U13.2 (I2)
- new net: U11.17 (IO1_4), U13.3 (I3)
- new net: U11.16 (IO1_3), U13.4 (I4)
- new net: U11.15 (IO1_2), U13.5 (I5)
- new net: U11.14 (IO1_1), U13.6 (I6)
- new net: U11.13 (IO1_0), U13.7 (I7)
- new net +12V: C15.1, C7.1, C8.1, D2.1 (K), D3.1 (K), J5.1 (Pin_1), Q2.3 (E), R12.2, TP4.1, U10.8 (V+), U9.3 (VI)
- new net A1: J2.3 (Pin_3), U3.10 (O7)
- new net A2: J3.3 (Pin_3), U4.10 (O7)
- new net A3: J7.3 (Pin_3), U7.10 (O7)
- new net A4: J8.3 (Pin_3), U8.10 (O7)
- new net A5: J10.3 (Pin_3), U12.10 (O7)
- new net A6: J11.3 (Pin_3), U13.10 (O7)
- new net B1: J2.4 (Pin_4), U3.11 (O6)
- new net B2: J3.4 (Pin_4), U4.11 (O6)
- new net B3: J7.4 (Pin_4), U7.11 (O6)
- new net B4: J8.4 (Pin_4), U8.11 (O6)
- new net B5: J10.4 (Pin_4), U12.11 (O6)
- new net B6: J11.4 (Pin_4), U13.11 (O6)
- new net C1: J2.5 (Pin_5), U3.12 (O5)
- new net C2: J3.5 (Pin_5), U4.12 (O5)
- new net C3: J7.5 (Pin_5), U7.12 (O5)
- new net C4: J8.5 (Pin_5), U8.12 (O5)
- new net C5: J10.5 (Pin_5), U12.12 (O5)
- new net C6: J11.5 (Pin_5), U13.12 (O5)
- new net D1: J2.6 (Pin_6), U3.13 (O4)
- new net D2: J3.6 (Pin_6), U4.13 (O4)
- new net D3: J7.6 (Pin_6), U7.13 (O4)
- new net D4: J8.6 (Pin_6), U8.13 (O4)
- new net D5: J10.6 (Pin_6), U12.13 (O4)
- new net D6: J11.6 (Pin_6), U13.13 (O4)
- new net E1: J2.7 (Pin_7), U3.14 (O3)
- new net E2: J3.7 (Pin_7), U4.14 (O3)
- new net E3: J7.7 (Pin_7), U7.14 (O3)
- new net E4: J8.7 (Pin_7), U8.14 (O3)
- new net E5: J10.7 (Pin_7), U12.14 (O3)
- new net E6: J11.7 (Pin_7), U13.14 (O3)
- new net F1: J2.8 (Pin_8), U3.15 (O2)
- new net F2: J3.8 (Pin_8), U4.15 (O2)
- new net F3: J7.8 (Pin_8), U7.15 (O2)
- new net F4: J8.8 (Pin_8), U8.15 (O2)
- new net F5: J10.8 (Pin_8), U12.15 (O2)
- new net F6: J11.8 (Pin_8), U13.15 (O2)
- new net G1: J2.9 (Pin_9), U3.16 (O1)
- new net G2: J3.9 (Pin_9), U4.16 (O1)
- new net G3: J7.9 (Pin_9), U7.16 (O1)
- new net G4: J8.9 (Pin_9), U8.16 (O1)
- new net G5: J10.9 (Pin_9), U12.16 (O1)
- new net G6: J11.9 (Pin_9), U13.16 (O1)
- new net VDD: J10.1 (Pin_1), J10.2 (Pin_2), J11.1 (Pin_1), J11.2 (Pin_2), J2.1 (Pin_1), J2.2 (Pin_2), J3.1 (Pin_1), J3.2 (Pin_2), J7.1 (Pin_1), J7.2 (Pin_2), J8.1 (Pin_1), J8.2 (Pin_2), Q2.2 (C), R13.1, R15.2, R17.1, TP1.1
- no-connect marks 0 -> 31
Other:
- moved on the sheet: U2, U5, Y1
