File: gps-seven-seg-clock-v2.kicad_pcb (KiCad board)
At the start: 4 copper layers, 100 x 50 mm, 74 parts, among them J1 SMA, J10 SM09B-GHS-TB, J11 SM09B-GHS-TB, J12 SM04B-GHS-TB, J2 SM09B-GHS-TB, J3 SM09B-GHS-TB, J4 ICSP, J5 XT30PW-M, J6 SM04B-GHS-TB, J7 SM09B-GHS-TB, J8 SM09B-GHS-TB, J9 SM06B-GHS-TB, Q2 MJD127, SW1 219-2LPST, U1 PCA9555PW, U10 AD8676xR, U11 PCA9555PW, U12 ULN2003A, U13 ULN2003A, U2 MAX-M10S, U3 ULN2003A, U4 ULN2003A, U5 ATmega328PB-A, U6 PCA9555PW, U7 ULN2003A, U8 ULN2003A, U9 NCP1117-3.3_TO252, Y1 8MHz

Commit message: sch and layout
Parts:
- removed D2, D3: B5819W, Diode_SMD:D_SOD-123
- removed J11: SM09B-GHS-TB, Connector_JST:JST_GH_SM09B-GHS-TB_1x09-1MP_P1.25mm_Horizontal
- removed J12: SM04B-GHS-TB, Connector_JST:JST_GH_SM04B-GHS-TB_1x04-1MP_P1.25mm_Horizontal
- removed SW1: 219-2LPST, Button_Switch_SMD:SW_DIP_SPSTx02_Slide_6.7x6.64mm_W8.61mm_P2.54mm_LowProfile
- removed U12, U13: ULN2003A, Package_SO:SOIC-16_3.9x9.9mm_P1.27mm
- removed Y1: 8MHz, Crystal:Resonator_SMD_Murata_CSTxExxV-3Pin_3.0x1.1mm_HandSoldering
- added C18: 0.1uF, Capacitor_SMD:C_0603_1608Metric, F.Cu at (207.0, 61.0)
- added C19: 0.1uF, Capacitor_SMD:C_0603_1608Metric, F.Cu at (163.8, 81.9)
- added C20: 0.1uF, Capacitor_SMD:C_0603_1608Metric, F.Cu at (216.1, 75.6)
- added C21: 0.1uF, Capacitor_SMD:C_0603_1608Metric, F.Cu at (156.8, 97.8)
- added C22: 100uF, Capacitor_SMD:C_1206_3216Metric_Pad1.33x1.80mm_HandSolder, F.Cu at (213.1, 138.4)
- added C23: 22uF, Capacitor_SMD:C_1206_3216Metric_Pad1.33x1.80mm_HandSolder, F.Cu at (174.5, 138.4)
- added C24: 22uF, Capacitor_SMD:C_1206_3216Metric_Pad1.33x1.80mm_HandSolder, F.Cu at (177.9, 138.4)
- added C25: 0.1uF, Capacitor_SMD:C_0603_1608Metric, F.Cu at (137.2, 90.2)
- added C26: 0.1uF, Capacitor_SMD:C_0603_1608Metric, F.Cu at (137.2, 106.2)
- added C27: 0.1uF, Capacitor_SMD:C_0603_1608Metric, F.Cu at (176.5, 60.3)
- added C28: 0.1uF, Capacitor_SMD:C_0603_1608Metric, F.Cu at (193.0, 60.3)
- added C29: 0.1uF, Capacitor_SMD:C_0603_1608Metric, F.Cu at (219.1, 116.3)
- added C30: 0.1uF, Capacitor_SMD:C_0603_1608Metric, F.Cu at (219.7, 99.7)
- added C31: 0.1uF, Capacitor_SMD:C_0603_1608Metric, F.Cu at (166.4, 119.4)
- added C32: 0.1uF, Capacitor_SMD:C_0603_1608Metric, F.Cu at (166.4, 116.2)
- added Q1: SiS176DN, Package_SO:Vishay_PowerPAK_1212-8_Single, F.Cu at (151.1, 135.9)
- added Q3: MMBT2222A, Package_TO_SOT_SMD:SOT-23, F.Cu at (149.2, 59.7)
- added R18: 100K, Resistor_SMD:R_0603_1608Metric, F.Cu at (145.4, 58.4)
- added R19: 2.2K, Resistor_SMD:R_0603_1608Metric, F.Cu at (149.9, 75.6)
- added R20: 0, Resistor_SMD:R_0603_1608Metric, F.Cu at (214.7, 131.1)
- added TP10: 5016, jannett_footprints:TestPoint_Keystone_5016_Vias, F.Cu at (219.7, 138.4)
- added TP11: 5016, jannett_footprints:TestPoint_Keystone_5016_Compact, F.Cu at (144.8, 75.6)
- added TP12: 5016, jannett_footprints:TestPoint_Keystone_5016_Compact, F.Cu at (144.8, 81.2)
- added TP13: 5016, jannett_footprints:TestPoint_Keystone_5016_Compact, F.Cu at (202.6, 66.8)
- added TP14: 5016, jannett_footprints:TestPoint_Keystone_5016_Compact, F.Cu at (209.6, 66.7)
- added TP5: 5016, jannett_footprints:TestPoint_Keystone_5016_Compact, F.Cu at (173.4, 101.6)
- added TP6: 5016, jannett_footprints:TestPoint_Keystone_5016_Vias, F.Cu at (159.4, 125.1)
- added TP7: 5016, jannett_footprints:TestPoint_Keystone_5016_Vias, F.Cu at (218.4, 66.7)
- added TP8: 5016, jannett_footprints:TestPoint_Keystone_5016_Compact, F.Cu at (214.6, 123.2)
- added TP9: 5016, jannett_footprints:TestPoint_Keystone_5016_Compact, F.Cu at (176.5, 123.8)
- C1, C10, C11, C2, C5, C6, C8, C9: value 0.1uF -> 22uF; footprint Capacitor_SMD:C_0603_1608Metric -> Capacitor_SMD:C_1206_3216Metric_Pad1.33x1.80mm_HandSolder
- C12: value 10uF -> 0.1uF
- C13: value 0.1uF -> 1nF
- C14: value 10uF -> 100pF
- C15: value 0.1uF -> 10nF
- C16: value 0.1uF -> 100uF; footprint Capacitor_SMD:C_0603_1608Metric -> Capacitor_SMD:C_1206_3216Metric_Pad1.33x1.80mm_HandSolder
- C3: value 10nF -> 22uF; footprint Capacitor_SMD:C_0603_1608Metric -> Capacitor_SMD:C_1206_3216Metric_Pad1.33x1.80mm_HandSolder
- C4: value 10uF -> 22uF; footprint Capacitor_SMD:C_0603_1608Metric -> Capacitor_SMD:C_1206_3216Metric_Pad1.33x1.80mm_HandSolder
- C7: value 100uF -> 22uF; footprint Capacitor_SMD:CP_Elec_6.3x5.4_Nichicon -> Capacitor_SMD:C_1206_3216Metric_Pad1.33x1.80mm_HandSolder
- D1: value LED -> CDBB345LR-HF; footprint LED_SMD:LED_0603_1608Metric_Pad1.05x0.95mm_HandSolder -> Diode_SMD:D_SMB
- J1: value SMA -> Conn_01x06; footprint Connector_Coaxial:SMA_Amphenol_132289_EdgeMount -> Connector_PinSocket_2.54mm:PinSocket_1x06_P2.54mm_Vertical
- J2: value SM09B-GHS-TB -> Conn_01x06; footprint Connector_JST:JST_GH_SM09B-GHS-TB_1x09-1MP_P1.25mm_Horizontal -> Connector_PinSocket_2.54mm:PinSocket_1x06_P2.54mm_Vertical
- J3: value SM09B-GHS-TB -> SM04B-GHS-TB; footprint Connector_JST:JST_GH_SM09B-GHS-TB_1x09-1MP_P1.25mm_Horizontal -> Connector_JST:JST_GH_SM04B-GHS-TB_1x04-1MP_P1.25mm_Horizontal
- J4: value ICSP -> SM04B-GHS-TB; footprint Connector_PinSocket_2.00mm:PinSocket_2x03_P2.00mm_Vertical -> Connector_JST:JST_GH_SM04B-GHS-TB_1x04-1MP_P1.25mm_Horizontal
- J5: value XT30PW-M -> SM09B-GHS-TB; footprint Connector_AMASS:AMASS_XT30PW-M_1x02_P2.50mm_Horizontal -> Connector_JST:JST_GH_SM09B-GHS-TB_1x09-1MP_P1.25mm_Horizontal
- J6: value SM04B-GHS-TB -> SM09B-GHS-TB; footprint Connector_JST:JST_GH_SM04B-GHS-TB_1x04-1MP_P1.25mm_Horizontal -> Connector_JST:JST_GH_SM09B-GHS-TB_1x09-1MP_P1.25mm_Horizontal
- J9: value SM06B-GHS-TB -> SM09B-GHS-TB; footprint Connector_JST:JST_GH_SM06B-GHS-TB_1x06-1MP_P1.25mm_Horizontal -> Connector_JST:JST_GH_SM09B-GHS-TB_1x09-1MP_P1.25mm_Horizontal
- L1: value 2.66 -> 10uH; footprint Inductor_SMD:L_0805_2012Metric_Pad1.15x1.40mm_HandSolder -> Inductor_SMD:L_Sunlord_MWSA1204S-100
- Q2: value MJD127 -> 2N7002; footprint Package_TO_SOT_SMD:TO-252-2 -> Package_TO_SOT_SMD:SOT-23
- R1: value 10 -> 0.1; footprint Resistor_SMD:R_0603_1608Metric -> Resistor_SMD:R_1206_3216Metric
- R10: value 100K -> 1K
- R11: value 10K -> 100K
- R12: value 4.99K -> 100K
- R14: value 1K -> 470; footprint Resistor_SMD:R_0603_1608Metric -> Resistor_SMD:R_1206_3216Metric
- R15, R7: value 1K -> 100K
- R16: value 10K -> 1K
- R17: value 470 -> 2.2K; footprint Resistor_SMD:R_1206_3216Metric -> Resistor_SMD:R_0603_1608Metric
- R2, R3: value 2.2K -> 69.8K
- R4: value 2.2K -> 1K
- R5: value 2.2K -> 40K
- R6: value 100K -> 10K
- R8: value 100K -> 0.05; footprint Resistor_SMD:R_0603_1608Metric -> Resistor_SMD:R_Shunt_Vishay_WSK2512_6332Metric_T2.21mm
- R9: value 100K -> 2.2K
- TP3: footprint jannett_footprints:TestPoint_Keystone_5016_Vias -> jannett_footprints:TestPoint_Keystone_5016_Compact
- TP4: value 5016 -> 20AWG Wire; footprint jannett_footprints:TestPoint_Keystone_5016_Vias -> TestPoint:TestPoint_THTPad_D2.0mm_Drill1.0mm
- U1: value PCA9555PW -> LM3488MM; footprint Package_SO:TSSOP-24_4.4x7.8mm_P0.65mm -> Package_SO:VSSOP-8_3x3mm_P0.65mm
- U10: value AD8676xR -> ULN2003A; footprint Package_SO:SOIC-8_3.9x4.9mm_P1.27mm -> Package_SO:SOIC-16_3.9x9.9mm_P1.27mm
- U11: value PCA9555PW -> ULN2003A; footprint Package_SO:TSSOP-24_4.4x7.8mm_P0.65mm -> Package_SO:SOIC-16_3.9x9.9mm_P1.27mm
- U2: value MAX-M10S -> ESP32 Dev Board; footprint RF_GPS:ublox_MAX -> jannett_footprints:ESP32_MODULE
- U5: value ATmega328PB-A -> ULN2003A; footprint Package_QFP:TQFP-32_7x7mm_P0.8mm -> Package_SO:SOIC-16_3.9x9.9mm_P1.27mm
- U7, U8: value ULN2003A -> PCA9555PW; footprint Package_SO:SOIC-16_3.9x9.9mm_P1.27mm -> Package_SO:TSSOP-24_4.4x7.8mm_P0.65mm
- U9: value NCP1117-3.3_TO252 -> ULN2003A; footprint Package_TO_SOT_SMD:TO-252-2 -> Package_SO:SOIC-16_3.9x9.9mm_P1.27mm
- moved H4 159.3 mm to (223.5, 147.3)
- moved U2 137.7 mm to (194.9, 125.7), turned to 180 degrees
- moved H3 128.5 mm to (132.1, 147.3)
- moved U5 126.3 mm to (217.2, 110.0), turned to 0 degrees
- moved L1 123.4 mm to (161.3, 141.0), turned to 180 degrees
- moved C2 121.1 mm to (161.6, 131.4)
- moved TP2 115.4 mm to (172.1, 148.6)
- moved C3 113.8 mm to (164.9, 131.4), turned to 90 degrees
- moved TP4 108.9 mm to (176.5, 143.5)
- moved C5 108.5 mm to (141.0, 137.8)
- moved J1 105.0 mm to (180.9, 90.8), turned to 180 degrees
- moved R8 104.9 mm to (153.7, 128.3), turned to 90 degrees
- moved J9 104.2 mm to (187.3, 54.6), turned to 180 degrees
- moved D1 103.2 mm to (148.6, 141.0)
- moved C4 102.2 mm to (168.3, 131.4), turned to 90 degrees
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Connections:
- C1 pad 1: +3.3V -> +5V
- C10 pad 1: /RESET -> /BULK_CAP
- C10 pad 2: Net-(J9-Pin_3) -> GND
- C11 pad 1: +3.3V -> /BULK_CAP
- C12 pad 1: +3.3V -> /DAC_FILT
- C13 pad 1: +3.3V -> /ISEN
- C14 pad 1: Net-(U10B--) -> /COMP
- C15 pad 1: +12V -> Net-(C15-Pad1)
- C16 pad 1: Net-(U10B-+) -> +3.3V
- C17 pad 1: Net-(C17-Pad1) -> /ADC0
- C17 pad 2: Net-(U10B--) -> GND
- C2 pad 1: +3.3V -> +5V
- C3 pad 1: Net-(C3-Pad1) -> +5V
- C4 pad 1: +3.3V -> +5V
- C5 pad 1: +3.3V -> VDD
- C6 pad 1: +3.3V -> VDD
- C7 pad 1: +12V -> /BULK_CAP
- C8 pad 1: +12V -> /BULK_CAP
- C9 pad 1: Net-(U10A-+) -> /BULK_CAP
- D1 pad 1: GND -> VDD
- D1 pad 2: Net-(D1-A) -> /SW
- J1 pad 1: Net-(J1-In) -> /1PPS
- J10 pad 3: /A5 -> /A6
- J10 pad 4: /B5 -> /B6
- J10 pad 5: /C5 -> /C6
- J10 pad 6: /D5 -> /D6
- J10 pad 7: /E5 -> /E6
- J10 pad 8: /F5 -> /F6
- J10 pad 9: /G5 -> /G6
- J2 pad 1: VDD -> GND
- J2 pad 2: VDD -> GND
- J2 pad 3: /A1 -> GND
- J2 pad 4: /B1 -> GND
- J2 pad 5: /C1 -> GND
- J2 pad 6: /D1 -> GND
- J3 pad 1: VDD -> +3.3V
- J3 pad 2: VDD -> /ADC0
- J3 pad 3: /A2 -> +3.3V
- J3 pad 4: /B2 -> /ADC1
- J4 pad 1: /MISO -> Net-(J4-Pin_1)
- J4 pad 2: +3.3V -> /LED_RTN
- J4 pad 3: /SCK -> Net-(J4-Pin_3)
- J4 pad 4: /MOSI -> /LED_RTN
- J5 pad 1: +12V -> VDD
- J5 pad 2: GND -> VDD
- J6 pad 1: /ADC0 -> VDD
- J6 pad 2: GND -> VDD
- J6 pad 3: /ADC1 -> /A3
- J6 pad 4: GND -> /B3
- J7 pad 3: /A3 -> /A5
- J7 pad 4: /B3 -> /B5
- J7 pad 5: /C3 -> /C5
- J7 pad 6: /D3 -> /D5
- J7 pad 7: /E3 -> /E5
- J7 pad 8: /F3 -> /F5
- J7 pad 9: /G3 -> /G5
- J8 pad 3: /A4 -> /A2
- J8 pad 4: /B4 -> /B2
- J8 pad 5: /C4 -> /C2
- J8 pad 6: /D4 -> /D2
- J8 pad 7: /E4 -> /E2
- J8 pad 8: /F4 -> /F2
- J8 pad 9: /G4 -> /G2
- J9 pad 1: +3.3V -> VDD
- J9 pad 2: Net-(D3-A) -> VDD
- J9 pad 3: Net-(J9-Pin_3) -> /A4
- J9 pad 4: /RX -> /B4
- J9 pad 5: /TX -> /C4
- J9 pad 6: GND -> /D4
- L1 pad 1: Net-(C3-Pad1) -> +5V
- L1 pad 2: Net-(J1-In) -> /SW
- Q2 pad 1: Net-(Q2-B) -> Net-(Q2-G)
- Q2 pad 2: VDD -> GND
- Q2 pad 3: +12V -> /BOOST_SHDN
- R1 pad 1: Net-(U2-VCC_RF) -> VDD
- R1 pad 2: Net-(C3-Pad1) -> /BULK_CAP
- R10 pad 1: /PWM9 -> /BOOST_SHDN_n
- R10 pad 2: Net-(U10A-+) -> Net-(Q2-G)
- R11 pad 1: Net-(U10A--) -> Net-(Q2-G)
- R11 pad 2: Net-(U10B--) -> GND
- R12 pad 1: Net-(U10B--) -> /ADC0
- R12 pad 2: +12V -> GND
- R13 pad 2: Net-(J12-Pin_3) -> Net-(J4-Pin_1)
- R14 pad 1: Net-(C17-Pad1) -> VDD
- R14 pad 2: Net-(Q2-B) -> Net-(J4-Pin_3)
- R15 pad 1: Net-(U10B-+) -> /ADC1
- R15 pad 2: VDD -> GND
- R16 pad 1: Net-(U10B-+) -> /COLONS
- R16 pad 2: GND -> Net-(Q3-B)
- R17 pad 1: VDD -> +3.3V
- R17 pad 2: Net-(J12-Pin_1) -> /SDA
- R2 pad 1: +3.3V -> VDD
- R2 pad 2: /SDA -> /FB
- R3 pad 1: +3.3V -> /FB
- R3 pad 2: /SCL -> /DAC_FILT
- R4 pad 1: +3.3V -> /DAC_FILT
- R4 pad 2: /SCL1 -> /DAC
- R5 pad 1: +3.3V -> /FA/SD
- R5 pad 2: /SDA1 -> /BOOST_SHDN
- R6 pad 1: /RESET -> /FB
- R6 pad 2: +3.3V -> GND
- R7 pad 1: /LED_INT -> +3.3V
- R7 pad 2: Net-(D1-A) -> /BOOST_SHDN
- R8 pad 1: /ADC0 -> /SRC
- R8 pad 2: +3.3V -> /ISEN
- R9 pad 1: /ADC1 -> /COMP
- R9 pad 2: +3.3V -> Net-(C15-Pad1)
- TP2 pad 1: GND -> +5V
- TP3 pad 1: +3.3V -> /FB
- TP4 pad 1: +12V -> +5V
- U1 pad 1: unconnected-(U1-~{INT}-Pad1) -> /ISEN
- U1 pad 2: GND -> /COMP
- U1 pad 3: GND -> /FB
- U1 pad 4: Net-(U1-IO0_0) -> GND
- U1 pad 5: Net-(U1-IO0_1) -> GND
- U1 pad 6: Net-(U1-IO0_2) -> /GATE
- U1 pad 7: Net-(U1-IO0_3) -> /FA/SD
- U1 pad 8: Net-(U1-IO0_4) -> +5V
- U10 pad 1: Net-(U10A--) -> Net-(U10-I1)
- U10 pad 2: Net-(U10A--) -> Net-(U10-I2)
- U10 pad 3: Net-(U10A-+) -> Net-(U10-I3)
- U10 pad 4: GND -> Net-(U10-I4)
- U10 pad 5: Net-(U10B-+) -> Net-(U10-I5)
- U10 pad 6: Net-(U10B--) -> Net-(U10-I6)
- U10 pad 7: Net-(C17-Pad1) -> Net-(U10-I7)
- U10 pad 8: +12V -> GND
- U11 pad 1: unconnected-(U11-~{INT}-Pad1) -> Net-(U11-I1)
- U11 pad 10: Net-(U11-IO0_6) -> /A6
- U11 pad 11: unconnected-(U11-IO0_7-Pad11) -> /B6
- U11 pad 12: GND -> /C6
- U11 pad 13: Net-(U11-IO1_0) -> /D6
- U11 pad 14: Net-(U11-IO1_1) -> /E6
- U11 pad 15: Net-(U11-IO1_2) -> /F6
- U11 pad 16: Net-(U11-IO1_3) -> /G6
- U11 pad 2: +3.3V -> Net-(U11-I2)
- U11 pad 3: GND -> Net-(U11-I3)
- U11 pad 4: Net-(U11-IO0_0) -> Net-(U11-I4)
- U11 pad 5: Net-(U11-IO0_1) -> Net-(U11-I5)
- U11 pad 6: Net-(U11-IO0_2) -> Net-(U11-I6)
- U11 pad 7: Net-(U11-IO0_3) -> Net-(U11-I7)
- U11 pad 8: Net-(U11-IO0_4) -> GND
- U11 pad 9: Net-(U11-IO0_5) -> VDD
- U2 pad 1: GND -> +3.3V
- U2 pad 10: GND -> unconnected-(U2-GPIO19-Pad10)
- U2 pad 11: Net-(J1-In) -> /SDA
- U2 pad 12: GND -> unconnected-(U2-GPIO3-Pad12)
- U2 pad 14: Net-(U2-VCC_RF) -> /SCL
- U2 pad 16: /SDA -> unconnected-(U2-EN-Pad16)
- U2 pad 17: /SCL -> unconnected-(U2-GPIO36-Pad17)
- U2 pad 2: /GPS_TX -> GND
- U2 pad 3: /GPS_RX -> unconnected-(U2-GPIO15-Pad3)
- U2 pad 4: /PPS -> unconnected-(U2-GPIO2-Pad4)
- U2 pad 5: unconnected-(U2-EXTINT-Pad5) -> Net-(U2-GPIO4)
- U2 pad 6: +3.3V -> /GPS_TXD
- U2 pad 7: +3.3V -> /GPS_RXD
- U2 pad 8: +3.3V -> /1PPS
- U3 pad 1: Net-(U1-IO0_6) -> Net-(U3-I1)
- U3 pad 2: Net-(U1-IO0_5) -> Net-(U3-I2)
- U3 pad 3: Net-(U1-IO0_4) -> Net-(U3-I3)
- U3 pad 4: Net-(U1-IO0_3) -> Net-(U3-I4)
- U3 pad 5: Net-(U1-IO0_2) -> Net-(U3-I5)
- U3 pad 6: Net-(U1-IO0_1) -> Net-(U3-I6)
- U3 pad 7: Net-(U1-IO0_0) -> Net-(U3-I7)
- U3 pad 9: unconnected-(U3-COM-Pad9) -> VDD
- U4 pad 1: Net-(U1-IO1_6) -> Net-(U4-I1)
- U4 pad 10: /A2 -> /A3
- U4 pad 11: /B2 -> /B3
- U4 pad 12: /C2 -> /C3
- U4 pad 13: /D2 -> /D3
- U4 pad 14: /E2 -> /E3
- U4 pad 15: /F2 -> /F3
- U4 pad 16: /G2 -> /G3
- U4 pad 2: Net-(U1-IO1_5) -> Net-(U4-I2)
- U4 pad 3: Net-(U1-IO1_4) -> Net-(U4-I3)
- U4 pad 4: Net-(U1-IO1_3) -> Net-(U4-I4)
- U4 pad 5: Net-(U1-IO1_2) -> Net-(U4-I5)
- U4 pad 6: Net-(U1-IO1_1) -> Net-(U4-I6)
- U4 pad 7: Net-(U1-IO1_0) -> Net-(U4-I7)
- U4 pad 9: unconnected-(U4-COM-Pad9) -> VDD
- U5 pad 1: /PPS -> Net-(U5-I1)
- U5 pad 10: unconnected-(U5-PD6-Pad10) -> /A5
- U5 pad 11: /LED_INT -> /B5
- U5 pad 12: unconnected-(U5-PB0-Pad12) -> /C5
- U5 pad 13: /PWM9 -> /D5
- U5 pad 14: unconnected-(U5-PB2-Pad14) -> /E5
- U5 pad 15: /MOSI -> /F5
- U5 pad 16: /MISO -> /G5
- U5 pad 2: unconnected-(U5-PD4-Pad2) -> Net-(U5-I2)
- U5 pad 3: /SDA1 -> Net-(U5-I3)
- U5 pad 4: +3.3V -> Net-(U5-I4)
- U5 pad 5: GND -> Net-(U5-I5)
- U5 pad 6: /SCL1 -> Net-(U5-I6)
- U5 pad 7: Net-(U5-XTAL1/PB6) -> Net-(U5-I7)
- U5 pad 8: Net-(U5-XTAL2/PB7) -> GND
- U5 pad 9: unconnected-(U5-PD5-Pad9) -> VDD
- U6 pad 10: Net-(U6-IO0_6) -> Net-(U3-I1)
- U6 pad 21: +3.3V -> GND
- U6 pad 4: Net-(U6-IO0_0) -> Net-(U3-I7)
- U6 pad 5: Net-(U6-IO0_1) -> Net-(U3-I6)
- U6 pad 6: Net-(U6-IO0_2) -> Net-(U3-I5)
- U6 pad 7: Net-(U6-IO0_3) -> Net-(U3-I4)
- U6 pad 8: Net-(U6-IO0_4) -> Net-(U3-I3)
- U6 pad 9: Net-(U6-IO0_5) -> Net-(U3-I2)
- U7 pad 1: Net-(U6-IO0_6) -> unconnected-(U7-~{INT}-Pad1)
- U7 pad 10: /A3 -> Net-(U4-I1)
- U7 pad 11: /B3 -> unconnected-(U7-IO0_7-Pad11)
- U7 pad 12: /C3 -> GND
- U7 pad 13: /D3 -> Net-(U10-I7)
- U7 pad 14: /E3 -> Net-(U10-I6)
- U7 pad 15: /F3 -> Net-(U10-I5)
- U7 pad 16: /G3 -> Net-(U10-I4)
- U7 pad 2: Net-(U6-IO0_5) -> GND
- U7 pad 3: Net-(U6-IO0_4) -> GND
- U7 pad 4: Net-(U6-IO0_3) -> Net-(U4-I7)
- U7 pad 5: Net-(U6-IO0_2) -> Net-(U4-I6)
- U7 pad 6: Net-(U6-IO0_1) -> Net-(U4-I5)
- U7 pad 7: Net-(U6-IO0_0) -> Net-(U4-I4)
- U7 pad 8: GND -> Net-(U4-I3)
- U7 pad 9: unconnected-(U7-COM-Pad9) -> Net-(U4-I2)
- U8 pad 1: Net-(U6-IO1_6) -> unconnected-(U8-~{INT}-Pad1)
- U8 pad 10: /A4 -> Net-(U5-I1)
- U8 pad 11: /B4 -> unconnected-(U8-IO0_7-Pad11)
- U8 pad 12: /C4 -> GND
- U8 pad 13: /D4 -> Net-(U11-I7)
- U8 pad 14: /E4 -> Net-(U11-I6)
- U8 pad 15: /F4 -> Net-(U11-I5)
- U8 pad 16: /G4 -> Net-(U11-I4)
- U8 pad 2: Net-(U6-IO1_5) -> +3.3V
- U8 pad 3: Net-(U6-IO1_4) -> GND
- U8 pad 4: Net-(U6-IO1_3) -> Net-(U5-I7)
- U8 pad 5: Net-(U6-IO1_2) -> Net-(U5-I6)
- U8 pad 6: Net-(U6-IO1_1) -> Net-(U5-I5)
- U8 pad 7: Net-(U6-IO1_0) -> Net-(U5-I4)
- U8 pad 8: GND -> Net-(U5-I3)
- U8 pad 9: unconnected-(U8-COM-Pad9) -> Net-(U5-I2)
- U9 pad 1: GND -> Net-(U6-IO1_6)
- U9 pad 2: +3.3V -> Net-(U6-IO1_5)
- U9 pad 3: +12V -> Net-(U6-IO1_4)
Routing:
- net /SCL1: track 64.2 -> 0.00 mm, vias 4 -> 0
- net /SDA1: track 64.0 -> 0.00 mm, vias 4 -> 0
- net GND: track 75.4 -> 23.8 mm, vias 97 -> 0
- net +3.3V: track 49.3 -> 0.00 mm, vias 11 -> 0
- net /DAC: track 0.00 -> 44.5 mm, vias 0 -> 1
- net /TX: track 40.2 -> 0.00 mm, vias 3 -> 0
- net Net-(J9-Pin_3): track 39.0 -> 0.00 mm, vias 2 -> 0
- net /RX: track 38.6 -> 0.00 mm, vias 3 -> 0
- net /SCL: track 38.0 -> 0.00 mm, vias 2 -> 0
- net /SDA: track 37.3 -> 0.00 mm, vias 2 -> 0
- net /PPS: track 34.2 -> 0.00 mm, vias 2 -> 0
- net /RESET: track 30.6 -> 0.00 mm, vias 1 -> 0
- net /ISEN: track 0.00 -> 30.4 mm, vias 0 -> 2
- net Net-(U10A-+): track 28.7 -> 0.00 mm
- net VDD: track 25.9 -> 0.00 mm, vias 14 -> 0
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- removed copper zone on B.Cu, net +12V
- removed copper zone on F.Cu, net +12V
- removed copper zone on In2.Cu, net +12V
- removed copper zone on F.Cu, net +3.3V
- removed copper zone on In2.Cu, net +3.3V
- removed copper zone on B.Cu, net GND
- removed copper zone on F.Cu, net GND
- removed copper zone on In2.Cu, net GND
- removed copper zone on B.Cu, net VDD
- removed copper zone on F.Cu, net VDD
Other:
- board size 100 x 50 mm -> 101.6 x 101.6 mm

Commit message: layout
Parts:
- moved C10 0.74 mm to (141.0, 123.7)
- moved C11 0.74 mm to (141.0, 120.4)
- moved C7 0.74 mm to (141.0, 133.7)
- moved C8 0.74 mm to (141.0, 130.4)
- moved C9 0.74 mm to (141.0, 127.0)
- moved R1 0.68 mm to (146.1, 128.5)
Routing:
- added copper zone on F.Cu, net +5V
- added copper zone on F.Cu, net /SW
- added copper zone on F.Cu, net VDD
Changed lines of the file:
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@@
 	(footprint "Capacitor_SMD:C_1206_3216Metric_Pad1.33x1.80mm_HandSolder"
 		(layer "F.Cu")
-		(at 140.335 130 180)
+		(at 140.97 130.381 180)
 		(descr "Capacitor SMD 1206 (3216 Metric), square (rectangular) end terminal, IPC-7351 nominal with elongated pad for handsoldering. (Body size source: IPC-SM-782 page 76, https://www.pcb-3d.com/wordpress/wp-content/uploads/ipc-sm-782a_amendment_1_and_2.pdf), generated with kicad-footprint-generator")
 		(tags "capacitor handsolder")
@@
 	(footprint "Capacitor_SMD:C_1206_3216Metric_Pad1.33x1.80mm_HandSolder"
 		(layer "F.Cu")
-		(at 140.335 120.015 180)
+		(at 140.97 120.396 180)
 		(descr "Capacitor SMD 1206 (3216 Metric), square (rectangular) end terminal, IPC-7351 nominal with elongated pad for handsoldering. (Body size source: IPC-SM-782 page 76, https://www.pcb-3d.com/wordpress/wp-content/uploads/ipc-sm-782a_amendment_1_and_2.pdf), generated with kicad-footprint-generator")
 		(tags "capacitor handsolder")
@@
 	(footprint "Capacitor_SMD:C_1206_3216Metric_Pad1.33x1.80mm_HandSolder"
 		(layer "F.Cu")
-		(at 140.335 126.65 180)
+		(at 140.97 127.031 180)
 		(descr "Capacitor SMD 1206 (3216 Metric), square (rectangular) end terminal, IPC-7351 nominal with elongated pad for handsoldering. (Body size source: IPC-SM-782 page 76, https://www.pcb-3d.com/wordpress/wp-content/uploads/ipc-sm-782a_amendment_1_and_2.pdf), generated with kicad-footprint-generator")
 		(tags "capacitor handsolder")
@@
 	(footprint "Capacitor_SMD:C_1206_3216Metric_Pad1.33x1.80mm_HandSolder"
 		(layer "F.Cu")
-		(at 140.335 123.3 180)
+		(at 140.97 123.681 180)
 		(descr "Capacitor SMD 1206 (3216 Metric), square (rectangular) end terminal, IPC-7351 nominal with elongated pad for handsoldering. (Body size source: IPC-SM-782 page 76, https://www.pcb-3d.com/wordpress/wp-content/uploads/ipc-sm-782a_amendment_1_and_2.pdf), generated with kicad-footprint-generator")
 		(tags "capacitor handsolder")
@@
 	(footprint "Resistor_SMD:R_1206_3216Metric"
 		(layer "F.Cu")
-		(at 145.415 128.27 180)
+		(at 146.05 128.524 180)
 		(descr "Resistor SMD 1206 (3216 Metric), square (rectangular) end terminal, IPC-7351 nominal, (Body size source: IPC-SM-782 page 72, https://www.pcb-3d.com/wordpress/wp-content/uploads/ipc-sm-782a_amendment_1_and_2.pdf), generated with kicad-footprint-generator")
 		(tags "resistor")
@@
 	(footprint "Capacitor_SMD:C_1206_3216Metric_Pad1.33x1.80mm_HandSolder"
 		(layer "F.Cu")
-		(at 140.335 133.35 180)
+		(at 140.97 133.731 180)
 		(descr "Capacitor SMD 1206 (3216 Metric), square (rectangular) end terminal, IPC-7351 nominal with elongated pad for handsoldering. (Body size source: IPC-SM-782 page 76, https://www.pcb-3d.com/wordpress/wp-content/uploads/ipc-sm-782a_amendment_1_and_2.pdf), generated with kicad-footprint-generator")
 		(tags "capacitor handsolder")
@@
 	)
 	(zone
+		(net 31)
+		(net_name "/SW")
+		(layer "F.Cu")
+		(hatch edge 0.5)
+		(priority 2)
+		(connect_pads yes
+			(clearance 0.5)
+		)
+		(min_thickness 0.25)
+		(filled_areas_thickness no)
+		(fill yes
+			(thermal_gap 0.5)
+			(thermal_bridge_width 0.5)
+		)
+		(polygon
+			(pts
+				(xy 149.225 135.255) (xy 156.21 135.255) (xy 156.21 135.89) (xy 158.115 137.795) (xy 158.115 144.78)
+				(xy 149.225 144.78)
+			)
+		)
+	)
+	(zone
+		(net 3)
+		(net_name "+5V")
+		(layer "F.Cu")
+		(hatch edge 0.5)
+		(priority 1)
+		(connect_pads yes
+			(clearance 0.5)
+		)
+		(min_thickness 0.25)
+		(filled_areas_thickness no)
+		(fill yes
+			(thermal_gap 0.5)
+			(thermal_bridge_width 0.5)
+		)
+		(polygon
+			(pts
+				(xy 180.975 140.335) (xy 183.515 140.335) (xy 183.515 151.13) (xy 158.115 151.13) (xy 158.115 137.795)
+				(xy 156.21 135.89) (xy 156.21 131.445) (xy 169.545 131.445) (xy 173.355 135.255) (xy 173.355 138.43)
+				(xy 179.07 138.43)
+			)
+		)
+	)
+	(zone
+		(net 8)
+		(net_name "VDD")
+		(layer "F.Cu")
+		(hatch edge 0.5)
+		(priority 3)
+		(connect_pads yes
+			(clearance 0.5)
+		)
+		(min_thickness 0.25)
+		(filled_areas_thickness no)
+		(fill yes
+			(thermal_gap 0.5)
+			(thermal_bridge_width 0.5)
+		)
+		(polygon
+			(pts
+				(xy 149.225 144.78) (xy 140.97 144.78) (xy 140.97 135.89) (xy 143.51 135.89) (xy 146.05 133.35)
+				(xy 146.05 124.46) (xy 144.78 123.19) (xy 144.78 116.205) (xy 145.415 115.57) (xy 150.495 115.57)
+				(xy 151.13 116.205) (xy 151.13 123.19) (xy 149.86 124.46) (xy 149.86 135.255) (xy 149.225 135.255)
+			)
+		)
+	)
+	(zone

Commit message: layout
Parts:
- added TP15: 5016, jannett_footprints:TestPoint_Keystone_5016_Vias, F.Cu at (134.6, 130.3)
- added TP16: 5016, jannett_footprints:TestPoint_Keystone_5016_Vias, F.Cu at (214.4, 134.9)
- added TP17: 5016, jannett_footprints:TestPoint_Keystone_5016_Vias, F.Cu at (169.4, 85.6)
- moved TP13 12.7 mm to (212.3, 58.7)
- moved TP10 9.30 mm to (214.4, 146.1)
- moved C20 7.83 mm to (223.9, 75.1)
- moved C18 7.78 mm to (199.3, 61.0)
- moved U8 7.74 mm to (217.9, 79.1)
- moved R17 7.71 mm to (148.7, 73.7)
- moved TP12 7.71 mm to (143.6, 73.6)
- moved J2 7.10 mm to (205.7, 76.7)
- moved J1 4.63 mm to (176.5, 89.4)
- moved R19 4.47 mm to (148.7, 79.9)
- moved TP11 4.47 mm to (143.6, 79.9)
- moved U7 4.13 mm to (157.7, 78.5)
- moved C19 3.53 mm to (161.7, 84.7)
- moved C16 3.01 mm to (173.2, 83.1)
- moved TP14 2.82 mm to (212.3, 66.3)
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Connections:
- U6 pad 22: /SCL1 -> /SCL
- U6 pad 23: /SDA1 -> /SDA
- U7 pad 22: /SCL1 -> /SCL
- U7 pad 23: /SDA1 -> /SDA
- U8 pad 22: /SCL1 -> /SCL
- U8 pad 23: /SDA1 -> /SDA
Routing:
- net /COLONS: track 0.00 -> 114.0 mm, vias 0 -> 1
- net /ADC0: track 0.00 -> 107.6 mm
- net /ADC1: track 0.00 -> 101.8 mm
- net GND: track 23.8 -> 86.7 mm, vias 0 -> 73
- net Net-(U10-I7): track 0.00 -> 57.5 mm
- net Net-(U10-I6): track 0.00 -> 55.3 mm
- net Net-(U10-I5): track 0.00 -> 53.1 mm
- net Net-(U10-I4): track 0.00 -> 50.9 mm
- net Net-(U10-I3): track 0.00 -> 48.5 mm
- net Net-(U10-I2): track 0.00 -> 46.0 mm
- net Net-(U10-I1): track 0.00 -> 43.6 mm
- net Net-(U5-I7): track 0.00 -> 41.0 mm
- net Net-(U5-I6): track 0.00 -> 38.9 mm
- net Net-(U5-I5): track 0.00 -> 36.6 mm
- net Net-(U5-I4): track 0.00 -> 34.3 mm
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- added copper zone on B.Cu, net +3.3V
- added copper zone on F.Cu, net +3.3V
- added copper zone on F.Cu, net /BULK_CAP
- added copper zone on F.Cu, net /SRC
- added copper zone on F.Cu, net GND
