File: gps-seven-seg-clock-v2.kicad_pcb (KiCad board)
At the start: 4 copper layers, 101.6 x 101.6 mm, 99 parts, among them J1 Conn_01x06, J10 SM09B-GHS-TB, J2 Conn_01x06, J3 SM04B-GHS-TB, J4 SM04B-GHS-TB, J5 SM09B-GHS-TB, J6 SM09B-GHS-TB, J7 SM09B-GHS-TB, J8 SM09B-GHS-TB, J9 SM09B-GHS-TB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

Commit message: gerbers and layout done
Parts:
- moved TP17 0.13 mm to (169.3, 85.6)
- moved C16 0.13 mm to (173.4, 83.1)
Routing:
- net /SDA: track 21.2 -> 187.5 mm, vias 0 -> 3
- net +3.3V: track 15.9 -> 176.5 mm, vias 7 -> 9
- net /SCL: track 18.8 -> 171.2 mm, vias 0 -> 4
- net /GPS_RST: track 0.00 -> 79.1 mm, vias 0 -> 1
- net /GPS_TXD: track 0.00 -> 69.1 mm
- net /GPS_RXD: track 0.00 -> 64.9 mm
- net /1PPS: track 7.25 -> 65.5 mm, vias 0 -> 1
- net +5V: track 3.94 -> 22.7 mm, vias 0 -> 2
- net /ISEN: track 30.4 -> 29.3 mm
Other:
- board text added: "1 3.3V 2 ADC0 3 3.3V 4 ADC1"
- board text added: "1 VCC 2 RTN 3 VCC 4 RTN"
- board text added: "1 VDD 2 VDD 3 a 4 b 5 c 6 d 7 e 8 f 9 g"
- board text added: "1PPS"
- board text added: "5V"
- board text added: "5V Pin"
- board text added: "ADC0"
- board text added: "ADC1"
- board text added: "BOOST"
- board text added: "DAC"
- board text added: "FB"
- board text added: "SCL"
- board text added: "SDA"
- board text added: "SHDN_n"
- board text added: "VCC"
- board text added: "Wire to"
- board text removed: "1 3.3V 2 VIN 3 RST 4 RX 5 TX 6 GND"
- board text removed: "1,2 Anodes 3-9 Cathodes"
- board text removed: "12V"
- board text removed: "4 GND 3 A1 2 GND 1 A0"
- board text removed: "4 GND 3 Anode 2 GND 1 Anode"
- board text removed: "Anode"
- board text removed: "MISO"
- board text removed: "MOSI"
- board text removed: "SCK"
