File: gps-seven-seg-clock-v2.kicad_sch (KiCad schematic)
At the start: 53 parts, among them J10 SM09B-GHS-TB, J11 SM09B-GHS-TB, J12 SM04B-GHS-TB, J2 SM09B-GHS-TB, J3 SM09B-GHS-TB, J5 XT30PW-M, J6 SM04B-GHS-TB, J7 SM09B-GHS-TB, J8 SM09B-GHS-TB, Q2 MJD127, U1 PCA9555PW, U10 AD8676xR, U11 PCA9555PW, U12 ULN2003A, U13 ULN2003A, U3 ULN2003A, U4 ULN2003A, U6 PCA9555PW, U7 ULN2003A, U8 ULN2003A, U9 NCP1117-3.3_TO252

Commit message: sch
Parts:
- removed C11, C15, C16, C17, C8, C9: 0.1uF, Capacitor_SMD:C_0603_1608Metric, symbol Device:C_Small
- removed C14: 10uF, Capacitor_SMD:C_0603_1608Metric, symbol Device:C_Small
- removed J5: XT30PW-M, Connector_AMASS:AMASS_XT30PW-M_1x02_P2.50mm_Horizontal, symbol Connector_Generic:Conn_01x02
- removed Q2: MJD127, Package_TO_SOT_SMD:TO-252-2, symbol Transistor_BJT:Q_PNP_Darlington_BCE
- removed R10: 100K, Resistor_SMD:R_0603_1608Metric, symbol Device:R_US
- removed R11, R16: 10K, Resistor_SMD:R_0603_1608Metric, symbol Device:R_US
- removed R12: 4.99K, Resistor_SMD:R_0603_1608Metric, symbol Device:R_US
- removed R14, R15: 1K, Resistor_SMD:R_0603_1608Metric, symbol Device:R_US
- removed TP4: 5016, jannett_footprints:TestPoint_Keystone_5016_Vias, symbol Connector:TestPoint
- removed U10: AD8676xR, Package_SO:SOIC-8_3.9x4.9mm_P1.27mm, symbol Amplifier_Operational:AD8676xR
- removed U9: NCP1117-3.3_TO252, Package_TO_SOT_SMD:TO-252-2, symbol Regulator_Linear:NCP1117-3.3_TO252
- added C2, C3: 100uF, Capacitor_SMD:CP_Elec_8x10.5, symbol Device:C_Polarized_US
- added C4: 1nF, Capacitor_SMD:C_0603_1608Metric, symbol Device:C_Small
- added D1: CD4148W, Diode_SMD:D_0805_2012Metric, symbol Diode:CD4148W
- added J1, J4: Conn_01x06, Connector_PinSocket_2.54mm:PinSocket_1x06_P2.54mm_Vertical, symbol Connector_Generic:Conn_01x06
- added L1: 10uH, symbol Device:L
- added Q1: SiS176DN, Package_SO:Vishay_PowerPAK_1212-8_Single, symbol Transistor_FET:SiS454DN
- added R1: 69.8K, Resistor_SMD:R_1206_3216Metric, symbol Device:R_US
- added R4: 10K, Resistor_SMD:R_1206_3216Metric, symbol Device:R_US
- added R5: 69.8K, Resistor_SMD:R_0603_1608Metric, symbol Device:R_US
- added R6: 4m, Resistor_SMD:R_1206_3216Metric, symbol Device:R_US
- added U2: ESP32 Dev Board, jannett_footprints:ESP32_MODULE, symbol jannett_symbols:ESP32_Module
- added U5: LM3488MM, Package_SO:VSSOP-8_3x3mm_P0.65mm, symbol Regulator_Controller:LM3478MM
Connections:
- net +3.3V: now also C2.1, C3.1, J1.5 (Pin_5), U2.1 (+3.3V); no longer D2.2 (A)
- net GND: now also C2.2, C3.2, C4.2, J1.2 (Pin_2), J4.1 (Pin_1), J4.2 (Pin_2), J4.3 (Pin_3), J4.4 (Pin_4), J4.5 (Pin_5), J4.6 (Pin_6), R4.2, R6.2, U2.2 (GND), U2.29 (GND), U5.4 (AGND), U5.5 (PGND); no longer TP2.1
- net SCL: now also U2.14 (GPIO22)
- net SDA: now also U2.11 (GPIO21)
- net VDD: now also D1.1 (K), R1.1; no longer TP1.1
- net +12V: no longer names the net of D2.1 (K)
- net +12V: no longer C7.1
- new net: D1.2 (A), L1.2, Q1.5 (D)
- new net: C4.1, Q1.1 (S), Q1.2 (S), Q1.3 (S), R6.1, U5.1 (I_{SEN})
- new net: R1.2, R4.1, R5.1, U5.3 (FB)
- new net: Q1.4 (G), U5.6 (DR)
- new net +5V: L1.1, U2.30 (VIN), U5.8 (V_{IN})
- new net 1PPS: J1.1 (Pin_1), U2.8 (GPIO5)
- new net DAC: R5.2, U2.23 (GPIO25)
- new net GPS_RST: J1.6 (Pin_6)
- new net GPS_RXD: J1.4 (Pin_4), U2.7 (GPIO17)
- new net GPS_TXD: J1.3 (Pin_3), U2.6 (GPIO16)
Other:
- moved on the sheet: C12, C7, D2, R2, R3, TP1, TP2

Commit message: sch and layout
Parts:
- removed C2, C3: 100uF, Capacitor_SMD:CP_Elec_8x10.5, symbol Device:C_Polarized_US
- removed C7: 100uF, Capacitor_SMD:CP_Elec_6.3x5.4_Nichicon, symbol Device:C_Polarized_US
- removed D1: CD4148W, Diode_SMD:D_0805_2012Metric, symbol Diode:CD4148W
- removed D2: B5819W, Diode_SMD:D_SOD-123, symbol Device:D_Schottky
- removed R6: 4m, Resistor_SMD:R_1206_3216Metric, symbol Device:R_US
- removed R8: 100K, Resistor_SMD:R_0603_1608Metric, symbol Device:R_US
- added C1, C10, C11, C2, C23, C24, C3, C4, C5, C6, C7, C8, C9: 22uF, Capacitor_SMD:C_1206_3216Metric_Pad1.33x1.80mm_HandSolder, symbol Device:C_Small
- added C14: 100pF, Capacitor_SMD:C_0603_1608Metric, symbol Device:C_Small
- added C15: 10nF, Capacitor_SMD:C_0603_1608Metric, symbol Device:C_Small
- added C16, C22: 100uF, Capacitor_SMD:C_1206_3216Metric_Pad1.33x1.80mm_HandSolder, symbol Device:C_Small
- added C17, C18, C25, C26, C27, C28, C29, C30, C31, C32: 0.1uF, Capacitor_SMD:C_0603_1608Metric, symbol Device:C_Small
- added D1: CDBB345LR-HF, Diode_SMD:D_SMB, symbol Diode:B240
- added Q2: 2N7002, Package_TO_SOT_SMD:SOT-23, symbol Transistor_FET:2N7002
- added Q3: MMBT2222A, Package_TO_SOT_SMD:SOT-23, symbol Transistor_BJT:MMBT2222A
- added R1: 0.1, Resistor_SMD:R_1206_3216Metric, symbol Device:R_US
- added R10, R16, R4: 1K, Resistor_SMD:R_0603_1608Metric, symbol Device:R_US
- added R11, R12, R15, R18, R7: 100K, Resistor_SMD:R_0603_1608Metric, symbol Device:R_US
- added R20: 0, Resistor_SMD:R_0603_1608Metric, symbol Device:R_US
- added R5: 40K, Resistor_SMD:R_0603_1608Metric, symbol Device:R_US
- added R8: 0.05, Resistor_SMD:R_Shunt_Vishay_WSK2512_6332Metric_T2.21mm, symbol Device:R_Shunt_US
- added TP10, TP6, TP7: 5016, jannett_footprints:TestPoint_Keystone_5016_Vias, symbol Connector:TestPoint
- added TP11, TP12, TP13, TP14, TP3, TP5, TP8, TP9: 5016, jannett_footprints:TestPoint_Keystone_5016_Compact, symbol Connector:TestPoint
- added TP4: 20AWG Wire, TestPoint:TestPoint_THTPad_D2.0mm_Drill1.0mm, symbol Connector:TestPoint
- C12: value 10uF -> 0.1uF
- L1: footprint (none) -> Inductor_SMD:L_Sunlord_MWSA1204S-100
- R2: renamed from R1; footprint Resistor_SMD:R_1206_3216Metric -> Resistor_SMD:R_0603_1608Metric
- R6: renamed from R4; footprint Resistor_SMD:R_1206_3216Metric -> Resistor_SMD:R_0603_1608Metric
- R9: value 100K -> 2.2K
- renumbered C4 to C13, C1 to C19, C6 to C20, C13 to C21, J4 to J1, J11 to J10, J1 to J2, J6 to J3, J12 to J4, J2 to J5, J7 to J6, J10 to J7, J3 to J8, J8 to J9, R17 to R13, R13 to R14, R2 to R17, R3 to R19, R5 to R3, U5 to U1, U8 to U10, U13 to U11, U7 to U4, U12 to U5, U1 to U6, U6 to U7, U11 to U8, U4 to U9
Connections:
- net +3.3V: now also J1.5 (Pin_5), J3.1 (Pin_1), J3.3 (Pin_3), C16.1, C22.1, R7.1, TP10.1; no longer C12.1, J2.5 (Pin_5), R9.2
- net +5V: now also TP2.1, C1.1, C2.1, C23.1, C24.1, C3.1, C31.1, C32.1, C4.1, TP4.1
- net 1PPS: now also J1.1 (Pin_1), TP8.1; no longer J2.1 (Pin_1)
- net ADC0: now also J3.2 (Pin_2), U2.21 (GPIO32), C17.1, R12.1, TP13.1; no longer J3.1 (Pin_1)
- net ADC1: now also J3.4 (Pin_4), U2.22 (GPIO33), C18.1, R15.1, TP14.1; no longer J3.3 (Pin_3), R9.1
- net DAC: now also R4.2, TP9.1; no longer R3.2
- net GND: now also J2.1 (Pin_1), J2.3 (Pin_3), J2.4 (Pin_4), J2.5 (Pin_5), J2.6 (Pin_6), C1.2, C10.2, C11.2, C14.2, C15.2, C16.2, C17.2, C18.2, C2.2, C22.2, C23.2, C24.2, C25.2, C26.2, C27.2, C28.2, C29.2, C3.2, C30.2, C31.2, C32.2, C4.2, C5.2, C6.2, C7.2, C8.2, C9.2, Q2.2 (S), Q3.2 (E), R11.2, R12.2, R15.2, R18.2, R8.3, R8.4, TP6.1, TP7.1; no longer J1.1 (Pin_1), J1.3 (Pin_3), J1.4 (Pin_4), J1.5 (Pin_5), J1.6 (Pin_6), J3.2 (Pin_2), J3.4 (Pin_4), J4.2 (Pin_2), J4.4 (Pin_4)
- net GPS_RST: now also J1.6 (Pin_6), R20.2; no longer J2.6 (Pin_6)
- net GPS_RXD: now also J1.4 (Pin_4); no longer J2.4 (Pin_4)
- net GPS_TXD: now also J1.3 (Pin_3); no longer J2.3 (Pin_3)
- net SCL: now also TP11.1
- net SDA: now also TP12.1
- net VDD: now also TP1.1, U10.9 (COM), U11.9 (COM), U3.9 (COM), U4.9 (COM), U5.9 (COM), U9.9 (COM), C25.1, C26.1, C27.1, C28.1, C29.1, C30.1, C5.1, C6.1, D1.1 (K), R1.1
- net SW: now reaches L1.2, Q1.5 (D)
- net SW: now also D1.2 (A)
- net SRC: now reaches Q1.1 (S), Q1.2 (S), Q1.3 (S)
- net SRC: now also R8.1; no longer C13.1, U1.1 (I_{SEN})
- net COMP: now reaches U1.2 (COMP)
- net COMP: now also R9.1, C14.1
- net FB: now reaches R2.2, R3.1, R6.1, U1.3 (FB)
- net FB: now also TP3.1
- net GATE: now reaches Q1.4 (G), U1.6 (DR)
- net FA/SD: now reaches U1.7 (FA/SD)
- net FA/SD: now also R5.1
- net BOOST_SHDN_n: now reaches U2.24 (GPIO26)
- net BOOST_SHDN_n: now also R10.1, TP5.1
- net COLONS: now reaches U2.25 (GPIO27)
- net COLONS: now also R16.1
- net at U2.5 (GPIO4): now also R20.1
- new net: Q2.1 (G), R10.2, R11.1
- new net: Q3.1 (B), R16.2, R18.1
- new net: C15.1, R9.2
- new net BOOST_SHDN: Q2.3 (D), R5.2, R7.2
- new net BULK_CAP: C10.1, C11.1, C7.1, C8.1, C9.1, R1.2
- new net DAC_FILT: C12.1, R3.2, R4.1
- new net ISEN: C13.1, R8.2, U1.1 (I_{SEN})
- new net LED_RTN: J4.2 (Pin_2), J4.4 (Pin_4), Q3.3 (C)
- no-connect marks 15 -> 9
Other:
- note added: "C3216X5R1V226M160AC"
- note added: "GRM31CR60J107KEA8L"
- note added: "HCM1A1305V3-100-R"
- moved on the sheet: C13, H1, H2, H3, H4, J1, J2, J3, J4, L1, Q1, R13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

Commit message: layout
Parts:
- added TP15, TP16, TP17: 5016, jannett_footprints:TestPoint_Keystone_5016_Vias, symbol Connector:TestPoint
Connections:
- net SCL1 is gone; now on net SCL: U6.22 (SCL), U7.22 (SCL), U8.22 (SCL)
- net SDA1 is gone; now on net SDA: U6.23 (SDA), U7.23 (SDA), U8.23 (SDA)
- net GND: now also TP15.1, TP16.1, TP17.1
